File: BaSHi-ZERO-1/REV_A/kicad/BaSHi-ZERO-1.kicad_sch (KiCad schematic)
At the start: 22 parts, among them J1 Conn_01x03, J2 1x02_Jumper, J3 1x02_Jumper, J4 Conn_01x08, J5 Conn_01x08, U1 AP63205WU, U2 74LVC1G07, U3 CMT8021N1L

Commit message: .
Parts:
- J4: footprint Connector_PinHeader_2.54mm:PinHeader_1x09_P2.54mm_Vertical -> Connector_PinSocket_2.54mm:PinSocket_1x09_P2.54mm_Vertical
Changed lines of the file:
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@@
 			)
 		)
-		(property "Footprint" "Connector_PinHeader_2.54mm:PinHeader_1x09_P2.54mm_Vertical"
+		(property "Footprint" "Connector_PinSocket_2.54mm:PinSocket_1x09_P2.54mm_Vertical"
 			(at 179.07 104.14 0)
 			(effects
